File: circuit/CounterDSP.sch (KiCad schematic (older format))
At the start: 9 parts, among them J1 CONN_01X02, J2 CONN_01X03, U1 dsPIC33FJ128GP802-I/SP, U2 TL072

Commit message: Pretty up schematics
Parts:
- U2: value TL072 -> TL972
Connections:
- net AMP renamed TO_DSP
Other:
- note added: "Virtual \nGround\n"
- moved on the sheet: C1, J2, R1, R2, U1, U2A
