File: newamp/_saved_nVamp.sch (KiCad schematic (older format))
At the start: 24 parts, among them J1 CONN_01X02, J2 CONN_01X03, J3 CONN_01X02, J4 CONN_01X02, U1 AD8428, U2 ADA4528, U3 ADA4528, U4 AD8428

Commit message: Make a better, 4 layer design for nVamp
Parts:
- added C10, C11: CP, Capacitors_THT:CP_Radial_D8.0mm_P3.50mm, symbol CP
- gave numbers to parts that had none: 6
Connections:
- net GND: now also C10.2, C11.1
- net VDD: now also C10.1
- net VEE: now also C11.2
Changed lines of the file:
@@
 $EndComp
 $Comp
-L C_Small C?
+L C_Small C8
 U 1 1 5A8445FB
 P 5900 2100
-F 0 "C?" H 5992 2146 50  0000 L CNN
+F 0 "C8" H 5992 2146 50  0000 L CNN
 F 1 "100n" H 5992 2055 50  0000 L CNN
 F 2 "Capacitors_SMD:C_0603_HandSoldering" H 5900 2100 50  0001 C CNN
@@
 $EndComp
 $Comp
-L C_Small C?
+L C_Small C9
 U 1 1 5A844634
 P 6050 2100
-F 0 "C?" H 6142 2146 50  0000 L CNN
+F 0 "C9" H 6142 2146 50  0000 L CNN
 F 1 "100n" H 6142 2055 50  0000 L CNN
 F 2 "Capacitors_SMD:C_0603_HandSoldering" H 6050 2100 50  0001 C CNN
@@
 $EndComp
 $Comp
-L C_Small C?
+L C_Small C7
 U 1 1 5A84466B
 P 5600 2100
-F 0 "C?" H 5692 2146 50  0000 L CNN
+F 0 "C7" H 5692 2146 50  0000 L CNN
 F 1 "100n" H 5692 2055 50  0000 L CNN
 F 2 "Capacitors_SMD:C_0603_HandSoldering" H 5600 2100 50  0001 C CNN
@@
 Connection ~ 5750 2200
 $Comp
-L C_Small C?
+L C_Small C4
 U 1 1 5A844791
 P 5050 2050
-F 0 "C?" H 5142 2096 50  0000 L CNN
+F 0 "C4" H 5142 2096 50  0000 L CNN
 F 1 "100n" H 5142 2005 50  0000 L CNN
 F 2 "Capacitors_SMD:C_0603_HandSoldering" H 5050 2050 50  0001 C CNN
@@
 $EndComp
 $Comp
-L C_Small C?
+L C_Small C5
 U 1 1 5A8447CF
 P 5200 2050
-F 0 "C?" H 5292 2096 50  0000 L CNN
+F 0 "C5" H 5292 2096 50  0000 L CNN
 F 1 "100n" H 5292 2005 50  0000 L CNN
 F 2 "Capacitors_SMD:C_0603_HandSoldering" H 5200 2050 50  0001 C CNN
@@
 $EndComp
 $Comp
-L C_Small C?
+L C_Small C6
 U 1 1 5A844814
 P 5350 2050
-F 0 "C?" H 5442 2096 50  0000 L CNN
+F 0 "C6" H 5442 2096 50  0000 L CNN
 F 1 "100n" H 5442 2005 50  0000 L CNN
 F 2 "Capacitors_SMD:C_0603_HandSoldering" H 5350 2050 50  0001 C CNN
@@
 Connection ~ 5200 2150
 Connection ~ 5050 2150
+$Comp
+L CP C10
+U 1 1 5A844CFD
+P 8300 2350
+F 0 "C10" H 8418 2396 50  0000 L CNN
+F 1 "CP" H 8418 2305 50  0000 L CNN
+F 2 "Capacitors_THT:CP_Radial_D8.0mm_P3.50mm" H 8338 2200 50  0001 C CNN
+F 3 "" H 8300 2350 50  0001 C CNN
+	1    8300 2350
+	1    0    0    -1
+$EndComp
+$Comp
+L CP C11
+U 1 1 5A844D5F
+P 8300 2650
+F 0 "C11" H 8418 2696 50  0000 L CNN
+F 1 "CP" H 8418 2605 50  0000 L CNN
+F 2 "Capacitors_THT:CP_Radial_D8.0mm_P3.50mm" H 8338 2500 50  0001 C CNN
+F 3 "" H 8300 2650 50  0001 C CNN
+	1    8300 2650
+	1    0    0    -1
+$EndComp
+$Comp
+L GND #PWR032
+U 1 1 5A844DAB
+P 8550 2500
+F 0 "#PWR032" H 8550 2250 50  0001 C CNN
+F 1 "GND" H 8555 2327 50  0000 C CNN
+F 2 "" H 8550 2500 50  0001 C CNN
+F 3 "" H 8550 2500 50  0001 C CNN
+	1    8550 2500
+	1    0    0    -1
+$EndComp
+$Comp
+L VEE #PWR033
+U 1 1 5A844DEA
+P 8300 2800
+F 0 "#PWR033" H 8300 2650 50  0001 C CNN
+F 1 "VEE" H 8318 2973 50  0000 C CNN
+F 2 "" H 8300 2800 50  0001 C CNN
+F 3 "" H 8300 2800 50  0001 C CNN
+	1    8300 2800
+	-1   0    0    1
+$EndComp
+$Comp
+L VDD #PWR034
+U 1 1 5A844E29
+P 8300 2200
+F 0 "#PWR034" H 8300 2050 50  0001 C CNN
+F 1 "VDD" H 8317 2373 50  0000 C CNN
+F 2 "" H 8300 2200 50  0001 C CNN
+F 3 "" H 8300 2200 50  0001 C CNN
+	1    8300 2200
+	1    0    0    -1
+$EndComp
+Wire Wire Line
+	8300 2500 8550 2500
 $EndSCHEMATC
